Commit message: Add Pilz planner, Cartesian pick, gripper fixes, and BT loop
Motion planning:
- Switch MoveIt kinematics solver from pick_ik to LMA
- Register Pilz Industrial Motion Planner alongside OMPL in MoveIt launch
- Add pilz_cartesian_limits.yaml for LIN/CIRC Cartesian velocity limits
- reach_location_server: use Pilz PTP as primary planner (deterministic,
  repeatable motion), fall back to OMPL only if PTP fails
- plan_to_pose: Pilz LIN straight-line Cartesian when goal flag is set

BT executor and action interface:
- Add cartesian bool field to ReachLocation.action goal
- CallAction BT node reads and forwards the cartesian flag
- bt_action.xml: cartesian="true" on pick move for straight-line approach
- bt_action.xml: gripper open speed 0.15->0.14 (avoids float32 limit error)
- bt_action.xml: release position 0.08->0.06 (avoids stall at 85mm limit)

Gripper result logic:
- result_callback: judge open/close success by actual reported position,
  not commanded target — fixes release always returning FAILURE when
  fingers stop just short of AT_DEST

BT loop:
- tick_function: remove timer cancel so BT retries on FAILURE and loops
  on SUCCESS indefinitely (home -> pick -> place cycle)

File: ur_driver/src/Universal_Robots_ROS2_Description/urdf/ur5e_workcell.urdf.xacro (robot description, xacro)
@@ -92,5 +92,5 @@
      script_sender_port="$(arg script_sender_port)"
      trajectory_port="$(arg trajectory_port)">
-    <origin xyz="0 0 0" rpy="0 0 0"/>
+    <origin xyz="0 0 0" rpy="0 0 ${pi}"/>
   </xacro:ur_robot>
   <xacro:table parent="world" prefix="$(arg prefix)">
@@ -109,5 +109,5 @@
     <parent link="world"/>
     <child link="frame"/>
-    <origin xyz="0 0 0" rpy="0 0 0"/>
+    <origin xyz="0 0 0" rpy="0 0 ${pi/2}"/>
   </joint>
   <link name="frame">
@@ -183,3 +183,12 @@
     </visual>
   </link>
+  <!-- Optical frame: Z-forward (depth), X-right, Y-down.                    -->
+  <!-- kinect_link +Y is the optical axis (thin face of body box).            -->
+  <!-- Roll −90° maps: optical Z → kinect_link Y, optical Y → kinect_link −Z -->
+  <joint name="kinect_to_rgb_optical" type="fixed">
+    <parent link="kinect_link"/>
+    <child link="kinect_rgb_optical_frame"/>
+    <origin xyz="0 0 0" rpy="-1.5707963 0 0"/>
+  </joint>
+  <link name="kinect_rgb_optical_frame"/>
 </robot>

File: ur_driver/src/Universal_Robots_ROS2_Driver/ur_moveit_config/srdf/ur_macro.srdf.xacro (robot description, xacro)
@@ -61,9 +61,7 @@
     <disable_collisions link1="frame" link2="${prefix}base_link"         reason="Adjacent"/>
     <disable_collisions link1="frame" link2="${prefix}base_link_inertia" reason="Adjacent"/>
-    <!-- Ceiling plate sits between shoulder (z=1.72m) and base_link_inertia  -->
-    <!-- (z=1.88m). base, shoulder, and upper_arm are always above or        -->
-    <!-- through it by design (robot hangs from the plate region).           -->
-    <!-- forearm, wrist and tool links remain checked so the plate           -->
-    <!-- constrains extreme elbow-forward/down configurations.               -->
+    <!-- Ceiling plate at z=1.75m. base_link_inertia (z=1.88m), shoulder_link  -->
+    <!-- (z=1.72m), and upper_arm_link (shoulder geometry overlaps plate) are  -->
+    <!-- structurally adjacent — disable all three to avoid false positives.   -->
     <disable_collisions link1="ceiling_plate" link2="${prefix}base_link"         reason="Adjacent"/>
     <disable_collisions link1="ceiling_plate" link2="${prefix}base_link_inertia" reason="Adjacent"/>
